File: Untitled.kicad_sch (KiCad schematic)
At the start: 0 parts

Commit message: feat: add dummy schematics + pcb
Parts:
- added J1: Screw Terminal Block 5.00 mm 2 pol, 2s_connectors:TerminalBlock_MaiXu_MX126-5.0-02P_1x02_P5.00mm, symbol 2s_connectors:Screw Terminal 5.00mm
- added R1: 47k_0805, Resistor_SMD:R_0805_2012Metric, symbol 2s_Resistor_0805:47k_0805
Connections:
- new net: J1.2 (Pin_2), R1.1
- new net GND: J1.1 (Pin_1), R1.2
