File: Untitled.kicad_pcb (KiCad board)
At the start: 2 copper layers, 0 parts

Commit message: feat: add dummy schematics + pcb
Parts:
- added J1: Screw Terminal Block 5.00 mm 2 pol, 2s_connectors:TerminalBlock_MaiXu_MX126-5.0-02P_1x02_P5.00mm, F.Cu at (144.2, 59.2)
- added R1: 47k_0805, Resistor_SMD:R_0805_2012Metric, F.Cu at (161.0, 62.1)
Routing:
- net GND: track 0.00 -> 17.5 mm
- net Net-(J1-Pin_2): track 0.00 -> 17.3 mm
Other:
- board outline added: 40 x 22.5 mm

Commit message: feat: use only major version if released
Other:
- board text added: "PCB Version: v${REVISION}"
- board text removed: "PCB Version: ${REVISION}"
Changed lines of the file:
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@@
 		(layer "Edge.Cuts")
 	)
-	(gr_text "PCB Version: ${REVISION}"
+	(gr_text "PCB Version: v${REVISION}"
 		(at 141.75 71.25 0)
 		(layer "F.SilkS")
