File: template.kicad_pcb (KiCad board)
At the start: 2 copper layers, 40 x 22.5 mm, 2 parts, among them J1 Screw Terminal Block 5.00 mm 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

Commit message: feat: add release workflow + add new text on PCB
Other:
- board text added: "${COMMENT9}"
- board text added: "Date: ${ISSUE_DATE}"
Changed lines of the file:
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@@
 	(paper "A4")
 	(title_block
+		(date "2025-11-09")
 		(rev "0.3.0-4-g86ce")
+		(comment 9 "githash")
 	)
 	(layers
@@
 	)
 	(gr_text "PCB Version: v${REVISION}"
-		(at 141.75 71.25 0)
+		(at 140.5 72 0)
 		(layer "F.SilkS")
 		(effects
+			(font
+				(size 1.5 1.5)
+				(thickness 0.3)
+				(bold yes)
+			)
+			(justify left bottom)
+		)
+	)
+	(gr_text "${COMMENT9}"
+		(at 174.75 53.25 0)
+		(layer "F.SilkS")
+		(effects
+			(font
+				(size 1.27 1.27)
+			)
+		)
+	)
+	(gr_text "Date: ${ISSUE_DATE}"
+		(at 141 54.75 0)
+		(layer "F.SilkS")
+		(effects
